Commit message: Kolmas kodutoo

File: src/my_r2d2/urdf/r2d2.urdf (robot description, URDF)
Before this commit: robot macroed, 5 links, 4 joints
Links:
- added link base_footprint
Joints:
- added joint base: type fixed, parent base_footprint, child base_link, origin xyz=0 0 ${bodylen/2+wheeldiam+0.1}

Commit message: Neljas kodutoo

File: src/my_r2d2/urdf/r2d2.urdf (robot description, URDF)
Before this commit: robot macroed, 6 links, 5 joints
Links:
- removed link lens
- added link eye; visual box size=0.0001 0.0001 0.0001
- added link lense; collision cylinder length=0.01 radius=0.07; visual cylinder length=0.01 radius=0.035
Joints:
- removed joint tolens
- added joint toeye: type fixed, parent lense, child eye, origin xyz=0 0 0 rpy=-1.5708 0 -1.5708
- added joint tolense: type fixed, parent box, child lense, origin xyz=0 0 0
